File: kicad/keyboard/keyboard.kicad_pcb (KiCad board)
At the start: 2 copper layers, 244 x 92 mm, 119 parts, among them SW1 SW_MX, SW10 SW_MX, SW11 SW_MX, SW12 SW_MX, SW13 SW_MX, SW14 SW_MX, SW15 SW_MX, SW16 SW_MX, SW17 SW_MX, SW18 SW_MX, SW19 SW_MX, SW2 SW_MX, SW20 SW_MX, SW21 SW_MX, SW22 SW_MX, SW23 SW_MX, SW24 SW_MX, SW25 SW_MX, SW26 SW_MX, SW27 SW_MX, SW28 SW_MX, SW29 SW_MX, SW3 SW_MX, SW30 SW_MX, SW31 SW_MX, SW32 SW_MX, SW33 SW_MX, SW34 SW_MX, SW35 SW_MX, SW36 SW_MX, SW37 SW_MX, SW38 SW_MX, SW39 SW_MX, SW4 SW_MX, SW40 SW_MX, SW41 SW_MX, SW42 SW_MX, SW43 SW_MX, SW44 SW_MX, SW45 SW_MX, SW46 SW_MX, SW47 SW_MX, SW48 SW_MX, SW49 SW_MX, SW5 SW_MX, SW50 SW_MX, SW51 SW_MX, SW52 SW_MX, SW53 SW_MX, SW54 SW_MX, SW55 SW_MX, SW56 SW_MX, SW57 SW_MX, SW58 SW_MX, SW59 SW_MX, SW6 SW_MX, SW7 SW_MX, SW8 SW_MX, SW9 SW_MX

Commit message: Change diode footprint
Parts:
- D1, D10, D11, D12, D13, D14, D15, D16, D17, D18, D19, D2, D20, D21, D22, D23, D24, D25, D26, D27, D28, D29, D3, D30, D31, D32, D33, D34, D35, D36, D37, D38, D39, D4, D40, D41, D42, D43, D44, D45, D46, D47, D48, D49, D5, D50, D51, D52, D53, D54, D55, D56, D57, D58, D59, D6, D7, D8, D9: footprint Diode_THT:D_DO-35_SOD27_P2.54mm_Vertical_KathodeUp -> Diode_THT:D_DO-35_SOD27_P7.62mm_Horizontal
- moved D1 2.50 mm to (47.8, 62.5)
- moved D12 2.50 mm to (47.8, 81.5)
- moved D23 2.50 mm to (47.8, 100.5)
- moved D47 2.50 mm to (47.8, 138.5)
- moved D34 2.46 mm to (47.8, 119.5)
- moved D5 0.25 mm to (107.2, 62.5)
Routing:
- net ROW0: track 264.4 -> 263.2 mm
- net ROW4: track 205.1 -> 204.1 mm
- net ROW3: track 203.5 -> 202.5 mm
- net ROW2: track 204.0 -> 203.0 mm
- net Net-(D47-A): track 12.3 -> 12.9 mm
- net Net-(D23-A): track 12.3 -> 12.9 mm
- net Net-(D12-A): track 12.3 -> 12.9 mm
- net Net-(D1-A): track 12.3 -> 12.9 mm
- net Net-(D34-A): track 12.3 -> 12.9 mm
- net Net-(D5-A): track 5.93 -> 5.30 mm
- net ROW1: track 235.4 -> 234.9 mm
