File: kicad/keyboard/keyboard.kicad_sch (KiCad schematic)
At the start: 119 parts, among them SW1 SW_MX, SW10 SW_MX, SW11 SW_MX, SW12 SW_MX, SW13 SW_MX, SW14 SW_MX, SW15 SW_MX, SW16 SW_MX, SW17 SW_MX, SW18 SW_MX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

Commit message: Change diode footprint
Parts:
- D1, D10, D11, D12, D13, D14, D15, D16, D17, D18, D19, D2, D20, D21, D22, D23, D24, D25, D26, D27, D28, D29, D3, D30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: footprint Diode_THT:D_DO-35_SOD27_P2.54mm_Vertical_KathodeUp -> Diode_THT:D_DO-35_SOD27_P7.62mm_Horizontal
